File: pcb/etapa_potencia.sch (KiCad schematic (older format))
At the start: 88 parts, among them Q1 MPSA56, Q10 MPSA06, Q11 MPSA06, Q12 MJE340, Q13 MJE340, Q14 MPSA56, Q15 MJE350, Q16 2sc3281, Q17 2sc3281, Q18 MJE350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

Commit message: 
Connections:
- net Entrada renamed Entrada+

Commit message: mas del kicad
Parts:
- added entrada-1: CONNECTOR, symbol CONNECTOR
Connections:
- net GND: now also entrada-1.1 (W)
Changed lines of the file:
@@
-EESchema Schematic File Version 2  date 02/05/2012 02:48:05 p.m.
+EESchema Schematic File Version 2  date mié 02 may 2012 15:04:55 ART
 LIBS:power
 LIBS:device
@@
 Comment4 ""
 $EndDescr
+Connection ~ 1050 4050
+$Comp
+L CONNECTOR entrada-1
+U 1 1 4FA17506
+P 1050 4050
+F 0 "entrada-1" V 1500 4000 70  0000 C CNN
+F 1 "CONNECTOR" V 1600 4050 70  0000 C CNN
+	1    1050 4050
+	0    -1   -1   0
+$EndComp
 Wire Wire Line
 	7000 4500 7400 4500

Commit message: mas del kicad
Changed lines of the file:
@@
-EESchema Schematic File Version 2  date mié 02 may 2012 15:04:55 ART
+EESchema Schematic File Version 2  date jue 03 may 2012 00:42:47 ART
 LIBS:power
 LIBS:device
@@
 Sheet 1 1
 Title ""
-Date "2 may 2012"
+Date "3 may 2012"
 Rev ""
 Comp ""
@@
 Connection ~ 5550 6900
 Text GLabel 650  4050 0    60   Input ~ 0
-Entrada-
+GND
 Text GLabel 650  5100 0    60   Input ~ 0
 Entrada+

Commit message: 
Parts:
- added R36: RVAR, symbol RVAR
Connections:
- net at C2.1, D2.2 (K), Q11.1 (E)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: now also R36.2; no longer R12.2
- new net: R12.2, R36.1

Commit message: Agregadas R nuevas; falta revisar grosores, componentes y pines
Parts:
- added R37, R38: R, symbol R
- Q11: value MPSA06 -> MJE340
Connections:
- net realim: now also R37.1, R38.1; no longer Q14.1 (E), Q20.1 (E)
- new net: Q20.1 (E), R37.2
- new net: Q14.1 (E), R38.2
Other:
- moved on the sheet: Q14, Q20

Commit message: muchas cosas mal en kicad
Parts:
- added C15, C16, C17: C, symbol C
- added R39: R, symbol R
Connections:
- net GND: now also C15.1, C16.1, C17.2
- net at 50V1.1 (W), C6.2, C8.2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: now also C15.2
- net at Q10.2 (B), Q8.1 (E), R8.1: no longer R7.2
- net at Q10.1 (E), R10.1: now also R7.2
- net at R16.1: now also D6.1 (A); no longer D6.2 (K)
- net at Q9.1 (E), R9.2: now also R39.2; no longer Q7.2 (B)
- net at D1.1 (A), R27.2, R28.2: no longer R29.1
- net at Q11.2 (B), R12.1, R28.1: no longer C2.2
- net at Q11.3 (C), R27.1: now also C2.2, R29.1
- net at Q16.1 (E), Q17.3 (C): now also D5.2 (K), R13.2
- net at 25V1.1 (W), D5.1 (A): now also C16.2
- net at -25V1.1 (W): now also D6.2 (K), C17.1; no longer D6.1 (A)
- new net: Q7.2 (B), R39.1
