File: Fuentes/pcb/pcb.sch (KiCad schematic (older format))
At the start: 21 parts, among them P1 entrada1, P2 entrada 2, P3 +50V, P4 -50V, P5 GND

Commit message: ultimo que hago en el dia
Parts:
- C1, C2, C3, C4: value C -> 100n
- C10, C11, C12, C5, C6, C7, C8, C9: value C -> 2200u
- D1, D2, D3, D4: value DIODE -> 6A10
Other:
- moved on the sheet: P5
Changed lines of the file:
@@
-EESchema Schematic File Version 2  date vie 01 jun 2012 00:05:45 ART
+EESchema Schematic File Version 2  date mié 20 jun 2012 17:24:06 ART
 LIBS:power
 LIBS:device
@@
 Sheet 1 1
 Title ""
-Date "1 jun 2012"
+Date "20 jun 2012"
 Rev ""
 Comp ""
@@
 $EndDescr
 Wire Wire Line
+	5050 1750 3200 1750
+Wire Wire Line
 	3200 1200 3200 1250
 Wire Wire Line
@@
 Connection ~ 4700 2300
 Connection ~ 4700 1200
-Wire Wire Line
-	3200 1750 5450 1750
 Connection ~ 3200 1750
 Wire Wire Line
@@
 Wire Wire Line
 	3650 1250 3650 1200
+Connection ~ 5050 1750
 $Comp
 L CONNECTOR P5
 U 1 1 4FC7AB52
-P 5450 1750
-F 0 "P5" H 5800 1850 70  0000 C CNN
-F 1 "GND" H 5700 1650 70  0000 C CNN
-	1    5450 1750
+P 5050 1750
+F 0 "P5" H 5400 1850 70  0000 C CNN
+F 1 "GND" H 5300 1650 70  0000 C CNN
+	1    5050 1750
 	1    0    0    -1
 $EndComp
@@
 P 3200 2000
 F 0 "C9" H 3250 2100 50  0000 L CNN
-F 1 "C" H 3250 1900 50  0000 L CNN
+F 1 "2200u" H 3250 1900 50  0000 L CNN
 	1    3200 2000
 	1    0    0    -1
@@
 P 3650 2000
 F 0 "C10" H 3700 2100 50  0000 L CNN
-F 1 "C" H 3700 1900 50  0000 L CNN
+F 1 "2200u" H 3700 1900 50  0000 L CNN
 	1    3650 2000
 	1    0    0    -1
@@
 P 4150 2000
 F 0 "C11" H 4200 2100 50  0000 L CNN
-F 1 "C" H 4200 1900 50  0000 L CNN
+F 1 "2200u" H 4200 1900 50  0000 L CNN
 	1    4150 2000
 	1    0    0    -1
@@
 P 4700 2000
 F 0 "C12" H 4750 2100 50  0000 L CNN
-F 1 "C" H 4750 1900 50  0000 L CNN
+F 1 "2200u" H 4750 1900 50  0000 L CNN
 	1    4700 2000
 	1    0    0    -1
@@
 P 4700 1450
 F 0 "C8" H 4750 1550 50  0000 L CNN
-F 1 "C" H 4750 1350 50  0000 L CNN
+F 1 "2200u" H 4750 1350 50  0000 L CNN
 	1    4700 1450
 	1    0    0    -1
@@
 P 4150 1450
 F 0 "C7" H 4200 1550 50  0000 L CNN
-F 1 "C" H 4200 1350 50  0000 L CNN
+F 1 "2200u" H 4200 1350 50  0000 L CNN
 	1    4150 1450
 	1    0    0    -1
@@
 P 3650 1450
 F 0 "C6" H 3700 1550 50  0000 L CNN
-F 1 "C" H 3700 1350 50  0000 L CNN
+F 1 "2200u" H 3700 1350 50  0000 L CNN
 	1    3650 1450
 	1    0    0    -1
@@
 P 3200 1450
 F 0 "C5" H 3250 1550 50  0000 L CNN
-F 1 "C" H 3250 1350 50  0000 L CNN
+F 1 "2200u" H 3250 1350 50  0000 L CNN
 	1    3200 1450
 	1    0    0    -1
@@
 P 1150 1450
 F 0 "C1" H 1200 1550 50  0000 L CNN
-F 1 "C" H 1200 1350 50  0000 L CNN
+F 1 "100n" H 1200 1350 50  0000 L CNN
 	1    1150 1450
 	1    0    0    -1
@@
 P 1150 2050
 F 0 "C2" H 1200 2150 50  0000 L CNN
-F 1 "C" H 1200 1950 50  0000 L CNN
+F 1 "100n" H 950 1900 50  0000 L CNN
 	1    1150 2050
 	1    0    0    -1
@@
 P 2200 2050
 F 0 "C4" H 2250 2150 50  0000 L CNN
-F 1 "C" H 2250 1950 50  0000 L CNN
+F 1 "100n" H 2250 1950 50  0000 L CNN
 	1    2200 2050
 	1    0    0    -1
@@
 P 2200 1450
 F 0 "C3" H 2250 1550 50  0000 L CNN
-F 1 "C" H 2250 1350 50  0000 L CNN
+F 1 "100n" H 2250 1350 50  0000 L CNN
 	1    2200 1450
 	1    0    0    -1
@@
 P 1900 2100
 F 0 "D4" H 1900 2200 40  0000 C CNN
-F 1 "DIODE" H 1900 2000 40  0000 C CNN
+F 1 "6A10" H 1900 2000 40  0000 C CNN
 	1    1900 2100
 	0    -1   -1   0
@@
 P 1450 2100
 F 0 "D2" H 1450 2200 40  0000 C CNN
-F 1 "DIODE" H 1450 2000 40  0000 C CNN
+F 1 "6A10" H 1450 2000 40  0000 C CNN
 	1    1450 2100
 	0    -1   -1   0
@@
 P 1450 1400
 F 0 "D1" H 1450 1500 40  0000 C CNN
-F 1 "DIODE" H 1450 1300 40  0000 C CNN
+F 1 "6A10" H 1450 1300 40  0000 C CNN
 	1    1450 1400
 	0    -1   -1   0
@@
 P 1900 1400
 F 0 "D3" H 1900 1500 40  0000 C CNN
-F 1 "DIODE" H 1900 1300 40  0000 C CNN
+F 1 "6A10" H 1900 1300 40  0000 C CNN
 	1    1900 1400
 	0    -1   -1   0
