File: preamp/preamp.sch (KiCad schematic (older format))
At the start: 32 parts, among them P1 CONNECTOR, P2 CONNECTOR, P3 CONNECTOR, P4 CONNECTOR, U1 TL082, U2 TL082

Commit message: ahora si
Parts:
- removed U1, U2: TL082, symbol TL082
- added P5: CONNECTOR, symbol CONNECTOR
- added U1, U2, U3: LM741, symbol LM741
Connections:
- no-connect marks 0 -> 6

Commit message: comienzo del analisis teorico
Parts:
- removed R1, R14, R6: R, symbol R
- added RV4: POT, symbol POT
Other:
- moved on the sheet: P5
Changed lines of the file:
@@
-EESchema Schematic File Version 2  date mié 04 jul 2012 22:03:06 ART
+EESchema Schematic File Version 2  date sáb 07 jul 2012 02:10:25 ART
 LIBS:power
 LIBS:device
@@
 Sheet 1 1
 Title ""
-Date "5 jul 2012"
+Date "7 jul 2012"
 Rev ""
 Comp ""
@@
 Comment4 ""
 $EndDescr
-NoConn ~ 3700 2000
-NoConn ~ 3800 2000
-NoConn ~ 5200 2100
-NoConn ~ 5300 2100
-NoConn ~ 6900 6850
-NoConn ~ 6800 6850
+Wire Wire Line
+	2150 600  1950 600
+Wire Wire Line
+	7250 1700 6200 1700
+Connection ~ 5500 6400
+Wire Wire Line
+	6300 6400 5500 6400
+Wire Wire Line
+	1500 800  1950 800
+Connection ~ 3850 800
+Wire Wire Line
+	3850 600  3850 800
+Wire Wire Line
+	3850 600  3200 600
 Wire Wire Line
 	6700 6950 6700 6850
@@
 	6550 4500 6500 4500
 Wire Wire Line
-	2850 4600 2850 4950
-Wire Wire Line
-	1500 1050 1500 800
+	2850 4950 2850 4600
+Wire Wire Line
+	1500 800  1500 1050
 Wire Wire Line
 	6800 1150 7000 1150
@@
 	2400 5750 6650 5750
 Wire Wire Line
-	7100 1700 7250 1700
-Wire Wire Line
 	7750 1700 7900 1700
 Connection ~ 5100 2400
 Wire Wire Line
 	5100 2400 5100 2500
-Wire Wire Line
-	5200 1300 5100 1300
 Connection ~ 6300 2400
 Connection ~ 6300 1700
 Wire Wire Line
-	6300 2400 6300 2200
+	6300 2200 6300 2400
 Wire Wire Line
 	2950 2200 2950 2400
@@
 Wire Wire Line
 	3200 1050 3200 1500
-Wire Wire Line
-	1500 800  2000 800
-Wire Wire Line
-	2950 900  2950 800
 Connection ~ 6700 6850
 Connection ~ 5500 4750
@@
 	4000 4000 4000 4200
 Wire Wire Line
-	4600 4200 4600 3850
+	4600 3850 4600 4200
 Connection ~ 2850 4000
 Wire Wire Line
@@
 	2250 4000 2250 4100
 Wire Wire Line
-	2850 3850 2850 4100
+	2850 4100 2850 3850
 Wire Wire Line
 	2250 4500 2250 4700
@@
 Connection ~ 2850 4700
 Wire Wire Line
-	4600 4700 4600 4950
+	4600 4950 4600 4700
 Wire Wire Line
 	4000 4600 4000 4800
@@
 	6650 5750 6650 5450
 Wire Wire Line
-	5550 4500 5450 4500
+	5450 4500 5550 4500
 Wire Wire Line
 	6100 4500 6050 4500
@@
 Wire Wire Line
 	3600 6150 5500 6150
-Wire Wire Line
-	5500 5300 5500 6550
-Wire Wire Line
-	5500 6550 6300 6550
 Connection ~ 5500 6150
 Wire Wire Line
-	6300 6350 6300 6400
-Wire Wire Line
-	2500 800  3300 800
+	6300 6400 6300 6350
 Wire Wire Line
 	3200 1700 2950 1700
@@
 	5350 1150 5300 1150
 Wire Wire Line
-	3800 800  5800 800
-Wire Wire Line
-	5800 800  5800 1700
+	5800 1700 5800 800
 Wire Wire Line
 	4700 1800 4700 2400
@@
 Wire Wire Line
 	2950 1700 2950 1300
-Wire Wire Line
-	3600 2000 3600 2050
-Wire Wire Line
-	6700 1700 6200 1700
-Wire Wire Line
-	2950 2400 7200 2400
-Wire Wire Line
-	7200 2400 7200 2200
 Wire Wire Line
 	7000 800  6800 800
@@
 	6700 6050 6700 5900
 Wire Wire Line
-	5500 4500 5500 4900
+	5500 4900 5500 4500
+Connection ~ 1900 800
+Wire Wire Line
+	1950 800  1950 600
+Wire Wire Line
+	2950 900  2950 750
+Wire Wire Line
+	5800 800  3850 800
+Wire Wire Line
+	5500 6400 5500 5300
+Wire Wire Line
+	2950 2400 6300 2400
+Wire Wire Line
+	2700 600  2550 600
+$Comp
+L C C8
+U 1 1 4FF7C4B1
+P 2350 600
+F 0 "C8" H 2400 700 50  0000 L CNN
+F 1 "C" H 2400 500 50  0000 L CNN
+	1    2350 600
+	0    -1   -1   0
+$EndComp
+$Comp
+L POT RV4
+U 1 1 4FF7C2C4
+P 2950 600
+F 0 "RV4" H 2950 500 50  0000 C CNN
+F 1 "POT" H 2950 600 50  0000 C CNN
+	1    2950 600
+	-1   0    0    1
+$EndComp
+NoConn ~ 3700 1200
+NoConn ~ 3800 1200
+NoConn ~ 5200 1300
+NoConn ~ 5300 1300
+NoConn ~ 6900 6850
+NoConn ~ 6800 6850
 $Comp
 L LM741 U3
@@
 F 1 "LM741" H 5350 1950 60  0000 C CNN
 	1    5200 1700
-	1    0    0    -1
+	1    0    0    1
 $EndComp
 $Comp
@@
 F 1 "LM741" H 3850 1850 60  0000 C CNN
 	1    3700 1600
-	1    0    0    -1
+	1    0    0    1
 $EndComp
 $Comp
 L CONNECTOR P5
 U 1 1 4FF4DBDD
-P 10100 900
-F 0 "P5" H 10450 1000 70  0000 C CNN
-F 1 "CONNECTOR" H 10450 800 70  0000 C CNN
-	1    10100 900
-	1    0    0    -1
-$EndComp
-$Comp
-L PWR_FLAG #FLG01
+P 8250 950
+F 0 "P5" H 8600 1050 70  0000 C CNN
+F 1 "CONNECTOR" H 8600 850 70  0000 C CNN
+	1    8250 950
+	1    0    0    -1
+$EndComp
+$Comp
+L PWR_FLAG #FLG2
 U 1 1 4FF4DBC4
 P 6800 1150
-F 0 "#FLG01" H 6800 1245 30  0001 C CNN
+F 0 "#FLG2" H 6800 1245 30  0001 C CNN
 F 1 "PWR_FLAG" H 6800 1330 30  0000 C CNN
 	1    6800 1150
@@
 $EndComp
 $Comp
-L PWR_FLAG #FLG02
+L PWR_FLAG #FLG1
 U 1 1 4FF4DBBF
 P 6800 800
-F 0 "#FLG02" H 6800 895 30  0001 C CNN
+F 0 "#FLG1" H 6800 895 30  0001 C CNN
 F 1 "PWR_FLAG" H 6800 980 30  0000 C CNN
 	1    6800 800
@@
 $EndComp
 $Comp
-L PWR_FLAG #FLG03
+L PWR_FLAG #FLG3
 U 1 1 4FF4DBB2
-P 10100 900
-F 0 "#FLG03" H 10100 995 30  0001 C CNN
-F 1 "PWR_FLAG" H 10100 1080 30  0000 C CNN
-	1    10100 900
-	1    0    0    -1
-$EndComp
-$Comp
-L GND #PWR04
+P 8250 950
+F 0 "#FLG3" H 8250 1045 30  0001 C CNN
+F 1 "PWR_FLAG" H 8250 1130 30  0000 C CNN
+	1    8250 950
+	1    0    0    -1
+$EndComp
+$Comp
+L GND #PWR3
 U 1 1 4FF4DBA0
-P 10100 900
-F 0 "#PWR04" H 10100 900 30  0001 C CNN
-F 1 "GND" H 10100 830 30  0001 C CNN
-	1    10100 900
+P 8250 950
+F 0 "#PWR3" H 8250 950 30  0001 C CNN
+F 1 "GND" H 8250 880 30  0001 C CNN
+	1    8250 950
 	1    0    0    -1
 $EndComp
@@
 Text Label 2400 5750 0    60   ~ 0
 1
-$Comp
-L R R14
-U 1 1 4FEE37CB
-P 7200 1950
-F 0 "R14" V 7280 1950 50  0000 C CNN
-F 1 "R" V 7200 1950 50  0000 C CNN
-	1    7200 1950
-	1    0    0    -1
-$EndComp
-$Comp
-L C C8
-U 1 1 4FEE37C1
-P 6900 1700
-F 0 "C8" H 6950 1800 50  0000 L CNN
-F 1 "C" H 6950 1600 50  0000 L CNN
-	1    6900 1700
-	0    1    1    0
-$EndComp
 Text Label 7850 1700 0    60   ~ 0
 1
 $Comp
-L GND #PWR05
+L GND #PWR1
 U 1 1 4FEE3676
 P 5100 2500
-F 0 "#PWR05" H 5100 2500 30  0001 C CNN
+F 0 "#PWR1" H 5100 2500 30  0001 C CNN
 F 1 "GND" H 5100 2430 30  0001 C CNN
 	1    5100 2500
 	1    0    0    -1
 $EndComp
-Text Label 5100 2200 2    60   ~ 0
+Text Label 5100 1300 2    60   ~ 0
 alim+
-Text Label 5200 1300 0    60   ~ 0
+Text Label 5100 2200 0    60   ~ 0
 alim-
-Text Label 3600 2050 2    60   ~ 0
+Text Label 3600 1150 2    60   ~ 0
 alim+
-Text Label 3600 1150 0    60   ~ 0
+Text Label 3600 2000 0    60   ~ 0
 alim-
 $Comp
@@
 $EndComp
 $Comp
-L R R6
-U 1 1 4FEE2FC6
-P 3550 800
-F 0 "R6" V 3630 800 50  0000 C CNN
-F 1 "R" V 3550 800 50  0000 C CNN
-	1    3550 800
-	0    1    1    0
-$EndComp
-$Comp
-L R R1
-U 1 1 4FEE2FB6
-P 2250 800
-F 0 "R1" V 2330 800 50  0000 C CNN
-F 1 "R" V 2250 800 50  0000 C CNN
-	1    2250 800
-	0    1    1    0
-$EndComp
-$Comp
 L R R4
 U 1 1 4FEE2F84
@@
 $EndComp
 $Comp
-L GND #PWR06
+L GND #PWR2
 U 1 1 4FEE2F30
-P 6300 6400
-F 0 "#PWR06" H 6300 6400 30  0001 C CNN
-F 1 "GND" H 6300 6330 30  0001 C CNN
-	1    6300 6400
-	1    0    0    -1
-$EndComp
+P 6300 6550
+F 0 "#PWR2" H 6300 6550 30  0001 C CNN
+F 1 "GND" H 6300 6480 30  0001 C CNN
+	1    6300 6550
+	1    0    0    -1
+$EndComp

Commit message: 
Parts:
- removed P1: CONNECTOR, symbol CONNECTOR
- added P1: Plug entrada, symbol CONN_2
Connections:
- wire segments 75 -> 76
Changed lines of the file:
@@
-EESchema Schematic File Version 2  date sáb 07 jul 2012 02:10:25 ART
+EESchema Schematic File Version 2  date sáb 07 jul 2012 14:32:06 ART
 LIBS:power
 LIBS:device
@@
 Comment4 ""
 $EndDescr
+$Comp
+L GND #PWR01
+U 1 1 4FF86E92
+P 1750 1550
+F 0 "#PWR01" H 1750 1550 30  0001 C CNN
+F 1 "GND" H 1750 1480 30  0001 C CNN
+	1    1750 1550
+	1    0    0    -1
+$EndComp
 Wire Wire Line
 	2150 600  1950 600
@@
 Connection ~ 5500 6400
 Wire Wire Line
-	6300 6400 5500 6400
-Wire Wire Line
-	1500 800  1950 800
+	5500 6400 6300 6400
+Wire Wire Line
+	1950 800  1500 800
 Connection ~ 3850 800
 Wire Wire Line
@@
 Wire Wire Line
 	2850 4950 2850 4600
-Wire Wire Line
-	1500 800  1500 1050
 Wire Wire Line
 	6800 1150 7000 1150
@@
 Connection ~ 6300 1700
 Wire Wire Line
-	6300 2200 6300 2400
-Wire Wire Line
-	2950 2200 2950 2400
+	6300 2400 6300 2200
+Wire Wire Line
+	2950 2400 2950 2200
 Wire Wire Line
 	4850 950  4700 950
@@
 	6700 3850 6650 3850
 Wire Wire Line
-	6650 3850 6650 3000
+	6650 3000 6650 3850
 Connection ~ 5500 4500
 Wire Wire Line
@@
 Connection ~ 4600 4000
 Wire Wire Line
-	4600 4000 4000 4000
+	4000 4000 4600 4000
 Wire Wire Line
 	4000 4000 4000 4200
@@
 Connection ~ 2850 4000
 Wire Wire Line
-	2850 4000 2250 4000
+	2250 4000 2850 4000
 Wire Wire Line
 	2250 4000 2250 4100
@@
 	5800 800  3850 800
 Wire Wire Line
-	5500 6400 5500 5300
-Wire Wire Line
-	2950 2400 6300 2400
+	5500 5300 5500 6400
+Wire Wire Line
+	6300 2400 2950 2400
 Wire Wire Line
 	2700 600  2550 600
+Wire Wire Line
+	1500 800  1500 1350
+Wire Wire Line
+	1500 1350 1750 1350
+$Comp
+L CONN_2 P1
+U 1 1 4FF86010
+P 2100 1450
+F 0 "P1" V 2050 1450 40  0000 C CNN
+F 1 "Plug entrada" V 2150 1450 40  0000 C CNN
+	1    2100 1450
+	1    0    0    -1
+$EndComp
 $Comp
 L C C8
@@
 $EndComp
 $Comp
-L PWR_FLAG #FLG2
+L PWR_FLAG #FLG02
 U 1 1 4FF4DBC4
 P 6800 1150
-F 0 "#FLG2" H 6800 1245 30  0001 C CNN
+F 0 "#FLG02" H 6800 1245 30  0001 C CNN
 F 1 "PWR_FLAG" H 6800 1330 30  0000 C CNN
 	1    6800 1150
@@
 $EndComp
 $Comp
-L PWR_FLAG #FLG1
+L PWR_FLAG #FLG03
 U 1 1 4FF4DBBF
 P 6800 800
-F 0 "#FLG1" H 6800 895 30  0001 C CNN
+F 0 "#FLG03" H 6800 895 30  0001 C CNN
 F 1 "PWR_FLAG" H 6800 980 30  0000 C CNN
 	1    6800 800
@@
 $EndComp
 $Comp
-L PWR_FLAG #FLG3
+L PWR_FLAG #FLG04
 U 1 1 4FF4DBB2
 P 8250 950
-F 0 "#FLG3" H 8250 1045 30  0001 C CNN
+F 0 "#FLG04" H 8250 1045 30  0001 C CNN
 F 1 "PWR_FLAG" H 8250 1130 30  0000 C CNN
 	1    8250 950
@@
 $EndComp
 $Comp
-L GND #PWR3
+L GND #PWR05
 U 1 1 4FF4DBA0
 P 8250 950
-F 0 "#PWR3" H 8250 950 30  0001 C CNN
+F 0 "#PWR05" H 8250 950 30  0001 C CNN
 F 1 "GND" H 8250 880 30  0001 C CNN
 	1    8250 950
@@
 	1    0    0    -1
 $EndComp
-$Comp
-L CONNECTOR P1
-U 1 1 4FEE38E3
-P 1500 1050
-F 0 "P1" H 1850 1150 70  0000 C CNN
-F 1 "CONNECTOR" H 1850 950 70  0000 C CNN
-	1    1500 1050
-	1    0    0    -1
-$EndComp
 Text Label 2400 5750 0    60   ~ 0
 1
@@
 1
 $Comp
-L GND #PWR1
+L GND #PWR06
 U 1 1 4FEE3676
 P 5100 2500
-F 0 "#PWR1" H 5100 2500 30  0001 C CNN
+F 0 "#PWR06" H 5100 2500 30  0001 C CNN
 F 1 "GND" H 5100 2430 30  0001 C CNN
 	1    5100 2500
@@
 $EndComp
 $Comp
-L GND #PWR2
+L GND #PWR07
 U 1 1 4FEE2F30
 P 6300 6550
-F 0 "#PWR2" H 6300 6550 30  0001 C CNN
+F 0 "#PWR07" H 6300 6550 30  0001 C CNN
 F 1 "GND" H 6300 6480 30  0001 C CNN
 	1    6300 6550

Commit message: empeze el pcb del pre
Parts:
- removed U1, U2, U3: LM741, symbol LM741
- added C10, C11, C12, C9: C, symbol C
- added R1, R6: R, symbol R
- added U1, U2: N35532, symbol N35532
- renumbered P2 to 20+1, P3 to 20-1
Connections:
- wire segments 76 -> 81
- no-connect marks 6 -> 0
Other:
- moved on the sheet: 20+1, 20-1, P4, R7

Commit message: pre conectado
Parts:
- renumbered P5 to ground1, P4 to salida1
Connections:
- net 1: no longer names the net of R15.1, R3.2, R9.2, RV3.1

Commit message: valores y version pasable del pre
Parts:
- C1: value C -> 47n
- C2: value C -> 22u
- C3, C5: value C -> 10n
- C4: value C -> 100p
- C6: value C -> 220
- C7: value C -> 2.2n
- C8: value C -> 220u
- R10: value R -> 47k
- R11: value R -> 15k
- R12: value R -> 10k
- R13, R4: value R -> 22k
- R15: value R -> 100
- R2, R3: value R -> 6k8
- R5: value R -> 68k
- R7: value R -> 680
- R8, R9: value R -> 2k2
Changed lines of the file:
@@
-EESchema Schematic File Version 2  date jue 19 jul 2012 00:48:19 ART
+EESchema Schematic File Version 2  date jue 19 jul 2012 23:11:59 ART
 LIBS:power
 LIBS:device
@@
 Sheet 1 1
 Title ""
-Date "19 jul 2012"
+Date "20 jul 2012"
 Rev ""
 Comp ""
@@
 P 2350 600
 F 0 "C8" H 2400 700 50  0000 L CNN
-F 1 "C" H 2400 500 50  0000 L CNN
+F 1 "220u" H 2400 500 50  0000 L CNN
 	1    2350 600
 	0    -1   -1   0
@@
 P 6000 1700
 F 0 "C6" H 6050 1800 50  0000 L CNN
-F 1 "C" H 6050 1600 50  0000 L CNN
+F 1 "220" H 6050 1600 50  0000 L CNN
 	1    6000 1700
 	0    1    1    0
@@
 P 5100 1150
 F 0 "C4" H 5150 1250 50  0000 L CNN
-F 1 "C" H 5150 1050 50  0000 L CNN
+F 1 "100p" H 4900 1050 50  0000 L CNN
 	1    5100 1150
 	0    -1   -1   0
@@
 P 2950 1100
 F 0 "C2" H 3000 1200 50  0000 L CNN
-F 1 "C" H 3000 1000 50  0000 L CNN
+F 1 "22u" H 3000 1000 50  0000 L CNN
 	1    2950 1100
 	1    0    0    -1
@@
 P 7500 1700
 F 0 "R15" V 7580 1700 50  0000 C CNN
-F 1 "R" V 7500 1700 50  0000 C CNN
+F 1 "100" V 7500 1700 50  0000 C CNN
 	1    7500 1700
 	0    1    1    0
@@
 P 5100 950
 F 0 "R10" V 5180 950 50  0000 C CNN
-F 1 "R" V 5100 950 50  0000 C CNN
+F 1 "47k" V 5100 950 50  0000 C CNN
 	1    5100 950
 	0    1    1    0
@@
 P 6300 1950
 F 0 "R13" V 6380 1950 50  0000 C CNN
-F 1 "R" V 6300 1950 50  0000 C CNN
+F 1 "22k" V 6300 1950 50  0000 C CNN
 	1    6300 1950
 	1    0    0    -1
@@
 P 4050 2150
 F 0 "R7" V 4130 2150 50  0000 C CNN
-F 1 "R" V 4050 2150 50  0000 C CNN
+F 1 "680" V 4050 2150 50  0000 C CNN
 	1    4050 2150
 	0    1    1    0
@@
 P 2950 1950
 F 0 "R4" V 3030 1950 50  0000 C CNN
-F 1 "R" V 2950 1950 50  0000 C CNN
+F 1 "22k" V 2950 1950 50  0000 C CNN
 	1    2950 1950
 	1    0    0    -1
@@
 P 5500 5100
 F 0 "C5" H 5550 5200 50  0000 L CNN
-F 1 "C" H 5550 5000 50  0000 L CNN
+F 1 "10n" H 5550 5000 50  0000 L CNN
 	1    5500 5100
 	1    0    0    -1
@@
 P 3350 4350
 F 0 "R5" V 3430 4350 50  0000 C CNN
-F 1 "R" H 3350 4350 50  0000 C CNN
+F 1 "68k" H 3350 4350 50  0000 C CNN
 	1    3350 4350
 	0    1    1    0
@@
 P 5200 4500
 F 0 "R11" V 5280 4500 50  0000 C CNN
-F 1 "R" H 5200 4500 50  0000 C CNN
+F 1 "15k" H 5200 4500 50  0000 C CNN
 	1    5200 4500
 	0    1    1    0
@@
 P 5800 4500
 F 0 "R12" V 5880 4500 50  0000 C CNN
-F 1 "R" H 5800 4500 50  0000 C CNN
+F 1 "10k" H 5800 4500 50  0000 C CNN
 	1    5800 4500
 	0    1    1    0
@@
 P 6300 4500
 F 0 "C7" H 6350 4600 50  0000 L CNN
-F 1 "C" H 6350 4400 50  0000 L CNN
+F 1 "2.2n" H 6350 4400 50  0000 L CNN
 	1    6300 4500
 	0    1    1    0
@@
 P 4000 4400
 F 0 "C3" H 4050 4500 50  0000 L CNN
-F 1 "C" H 4050 4300 50  0000 L CNN
+F 1 "10n" H 4050 4300 50  0000 L CNN
 	1    4000 4400
 	1    0    0    -1
@@
 P 2250 4300
 F 0 "C1" H 2300 4400 50  0000 L CNN
-F 1 "C" H 2300 4200 50  0000 L CNN
+F 1 "47n" H 2300 4200 50  0000 L CNN
 	1    2250 4300
 	1    0    0    -1
@@
 P 4600 5200
 F 0 "R9" V 4680 5200 50  0000 C CNN
-F 1 "R" V 4600 5200 50  0000 C CNN
+F 1 "2k2" V 4600 5200 50  0000 C CNN
 	1    4600 5200
 	1    0    0    -1
@@
 P 4600 3600
 F 0 "R8" V 4680 3600 50  0000 C CNN
-F 1 "R" V 4600 3600 50  0000 C CNN
+F 1 "2k2" V 4600 3600 50  0000 C CNN
 	1    4600 3600
 	1    0    0    -1
@@
 P 2850 5200
 F 0 "R3" V 2930 5200 50  0000 C CNN
-F 1 "R" V 2850 5200 50  0000 C CNN
+F 1 "6k8" V 2850 5200 50  0000 C CNN
 	1    2850 5200
 	1    0    0    -1
@@
 P 2850 3600
 F 0 "R2" V 2930 3600 50  0000 C CNN
-F 1 "R" V 2850 3600 50  0000 C CNN
+F 1 "6k8" V 2850 3600 50  0000 C CNN
 	1    2850 3600
 	1    0    0    -1
